File: Hub_USB_Raspberry_Pi_Zero_2W/USB.kicad_sch (KiCad schematic)
At the start: 5 parts, among them J2 USB_C_Receptacle_USB2.0_16P, U2 USBLC6-2SC6

Commit message: Update kicad HUB
Changed lines of the file:
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@@
 	)
 	(junction
-		(at 62.23 25.4)
+		(at 55.88 25.4)
 		(diameter 0)
 		(color 0 0 0 0)
@@
 	(wire
 		(pts
-			(xy 62.23 22.86) (xy 62.23 25.4)
+			(xy 55.88 22.86) (xy 55.88 25.4)
 		)
 		(stroke
@@
 	(wire
 		(pts
-			(xy 59.69 25.4) (xy 62.23 25.4)
-		)
-		(stroke
-			(width 0)
-			(type default)
-		)
-	)
-	(wire
-		(pts
 			(xy 69.85 44.45) (xy 73.66 44.45)
 		)
@@
 	(wire
 		(pts
-			(xy 85.09 46.99) (xy 91.44 46.99)
-		)
-		(stroke
-			(width 0)
-			(type default)
-		)
-	)
-	(wire
-		(pts
-			(xy 62.23 25.4) (xy 62.23 38.1)
+			(xy 90.17 46.99) (xy 91.44 46.99)
+		)
+		(stroke
+			(width 0)
+			(type default)
+		)
+	)
+	(wire
+		(pts
+			(xy 55.88 25.4) (xy 55.88 38.1)
 		)
 		(stroke
@@
 	(wire
 		(pts
-			(xy 62.23 38.1) (xy 54.61 38.1)
+			(xy 55.88 38.1) (xy 54.61 38.1)
 		)
 		(stroke
@@
 		(pts
 			(xy 59.69 57.15) (xy 62.23 57.15)
+		)
+		(stroke
+			(width 0)
+			(type default)
+		)
+	)
+	(wire
+		(pts
+			(xy 55.88 25.4) (xy 59.69 25.4)
 		)
 		(stroke
@@
 		)
 	)
-	(label "V_USB"
-		(at 62.23 38.1 180)
-		(effects
-			(font
-				(size 1.27 1.27)
-			)
-			(justify right bottom)
-		)
-	)
 	(label "D+"
 		(at 96.52 55.88 0)
@@
 	(label "D-"
 		(at 62.23 52.07 0)
-		(effects
-			(font
-				(size 1.27 1.27)
-			)
-			(justify left bottom)
-		)
-	)
-	(label "V_USB"
-		(at 85.09 46.99 0)
 		(effects
 			(font
@@
 		(shape input)
 		(at 86.36 53.34 180)
+		(effects
+			(font
+				(size 1.27 1.27)
+			)
+			(justify right)
+		)
+	)
+	(hierarchical_label "V_USB"
+		(shape input)
+		(at 55.88 38.1 0)
+		(effects
+			(font
+				(size 1.27 1.27)
+			)
+			(justify left)
+		)
+	)
+	(hierarchical_label "V_USB"
+		(shape input)
+		(at 90.17 46.99 180)
 		(effects
 			(font
@@
 		(dnp no)
 		(property "Reference" "C5"
-			(at 51.816 27.178 0)
+			(at 62.738 26.924 0)
 			(effects
 				(font
@@
 		)
 		(property "Value" "100uF"
-			(at 49.276 28.956 0)
+			(at 61.468 28.702 0)
 			(effects
 				(font
@@
 	(symbol
 		(lib_id "power:+5V")
-		(at 62.23 22.86 0)
+		(at 55.88 22.86 0)
 		(unit 1)
 		(exclude_from_sim no)
@@
 		(fields_autoplaced yes)
 		(property "Reference" "#PWR01"
-			(at 62.23 26.67 0)
+			(at 55.88 26.67 0)
 			(effects
 				(font
@@
 		)
 		(property "Value" "+5V"
-			(at 62.23 17.78 0)
+			(at 55.88 17.78 0)
 			(effects
 				(font
@@
 		)
 		(property "Footprint" ""
-			(at 62.23 22.86 0)
+			(at 55.88 22.86 0)
 			(effects
 				(font
@@
 		)
 		(property "Datasheet" ""
-			(at 62.23 22.86 0)
+			(at 55.88 22.86 0)
 			(effects
 				(font
@@
 		)
 		(property "Description" "Power symbol creates a global label with name \"+5V\""
-			(at 62.23 22.86 0)
-			(effects
-				(font
+			(at 55.88 22.86 0)
+			(effects
+				(font
