File: Hub_USB_Raspberry_Pi_Zero_2W/USB0.kicad_sch (KiCad schematic)
At the start: 5 parts, among them J2 USB_C_Receptacle_USB2.0_16P, U2 USBLC6-2SC6

Commit message: CB avançage
Parts:
- removed C6: 100uF, Capacitor_SMD:C_0603_1608Metric, symbol Device:C_Small
- removed J2: USB_C_Receptacle_USB2.0_16P, Connector_USB:USB_C_Receptacle_GCT_USB4105-xx-A_16P_TopMnt_Horizontal, symbol Connector:USB_C_Receptacle_USB2.0_16P
- removed R300, R400: 5.1k, Resistor_SMD:R_0603_1608Metric, symbol Device:R_Small
- removed U2: USBLC6-2SC6, Package_TO_SOT_SMD:SOT-23-6, symbol Power_Protection:USBLC6-2SC6
- added C5: 100uF, Capacitor_SMD:C_0603_1608Metric, symbol Device:C_Small
- added J1: USB_C_Receptacle_USB2.0_16P, Connector_USB:USB_C_Receptacle_GCT_USB4105-xx-A_16P_TopMnt_Horizontal, symbol Connector:USB_C_Receptacle_USB2.0_16P
- added R100, R110: 5.1k, Resistor_SMD:R_0603_1608Metric, symbol Device:R_Small
- added U1: USBLC6-2SC6, Package_TO_SOT_SMD:SOT-23-6, symbol Power_Protection:USBLC6-2SC6
Connections:
- net +5V: now also C5.1, J1.A4 (VBUS), J1.A9 (VBUS), J1.B4 (VBUS), J1.B9 (VBUS), U1.5 (VBUS)
- net D+: now also J1.A6 (D+), J1.B6 (D+), U1.4 (I/O2)
- net D-: now also J1.A7 (D-), J1.B7 (D-), U1.6 (I/O1)
- net GND: now also C5.2, J1.A1 (GND), J1.A12 (GND), J1.B1 (GND), J1.B12 (GND), J1.S1 (SHIELD), R100.2, R110.2, U1.2 (GND)
- net USB_DM: now also U1.3 (I/O2)
- net USB_DP: now also U1.1 (I/O1)
- new net: J1.A5 (CC1), R100.1
- new net: J1.B5 (CC2), R110.1
