File: 04_Electronique/Kicad_Project/Hub_USB_Raspberry_Pi_Zero_2W/USB.kicad_sch (KiCad schematic)
At the start: 5 parts, among them J2 USB_C_Receptacle_USB2.0_16P, U2 USBLC6-2SC6

Commit message: Finalisation premier PCB
Parts:
- renumbered C6 to C8, J2 to J4, R300 to R10, R400 to R11, U2 to U4
Changed lines of the file:
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@@
 		(dnp no)
 		(fields_autoplaced yes)
-		(property "Reference" "#PWR02"
+		(property "Reference" "#PWR?"
 			(at 55.88 26.67 0)
 			(effects
@@
 				(path "/7e321a74-9d7c-485f-8c03-6a7893ec6c14/7e15107b-ac9e-4ac1-975d-b2dcf8c4df08"
 					(reference "#PWR0101")
+					(unit 1)
+				)
+				(path "/7e321a74-9d7c-485f-8c03-6a7893ec6c14/a8302038-da8a-47d3-9e0b-3649230cd28e"
+					(reference "#PWR?")
 					(unit 1)
 				)
@@
 		(dnp no)
 		(fields_autoplaced yes)
-		(property "Reference" "U2"
+		(property "Reference" "U?"
 			(at 93.0911 45.72 0)
 			(effects
@@
 				(path "/7e321a74-9d7c-485f-8c03-6a7893ec6c14/7e15107b-ac9e-4ac1-975d-b2dcf8c4df08"
 					(reference "U3")
+					(unit 1)
+				)
+				(path "/7e321a74-9d7c-485f-8c03-6a7893ec6c14/a8302038-da8a-47d3-9e0b-3649230cd28e"
+					(reference "U?")
 					(unit 1)
 				)
@@
 		(dnp no)
 		(fields_autoplaced yes)
-		(property "Reference" "#PWR06"
+		(property "Reference" "#PWR?"
 			(at 91.44 67.31 0)
 			(effects
@@
 				(path "/7e321a74-9d7c-485f-8c03-6a7893ec6c14/7e15107b-ac9e-4ac1-975d-b2dcf8c4df08"
 					(reference "#PWR0105")
+					(unit 1)
+				)
+				(path "/7e321a74-9d7c-485f-8c03-6a7893ec6c14/a8302038-da8a-47d3-9e0b-3649230cd28e"
+					(reference "#PWR?")
 					(unit 1)
 				)
@@
 		(on_board yes)
 		(dnp no)
-		(property "Reference" "C6"
+		(property "Reference" "C?"
 			(at 62.738 26.924 0)
 			(effects
@@
 				(path "/7e321a74-9d7c-485f-8c03-6a7893ec6c14/7e15107b-ac9e-4ac1-975d-b2dcf8c4df08"
 					(reference "C7")
+					(unit 1)
+				)
+				(path "/7e321a74-9d7c-485f-8c03-6a7893ec6c14/a8302038-da8a-47d3-9e0b-3649230cd28e"
+					(reference "C?")
 					(unit 1)
 				)
@@
 		(dnp no)
 		(fields_autoplaced yes)
-		(property "Reference" "#PWR05"
+		(property "Reference" "#PWR?"
 			(at 73.66 50.8 0)
 			(effects
@@
 				(path "/7e321a74-9d7c-485f-8c03-6a7893ec6c14/7e15107b-ac9e-4ac1-975d-b2dcf8c4df08"
 					(reference "#PWR0104")
+					(unit 1)
+				)
+				(path "/7e321a74-9d7c-485f-8c03-6a7893ec6c14/a8302038-da8a-47d3-9e0b-3649230cd28e"
+					(reference "#PWR?")
 					(unit 1)
 				)
@@
 		(dnp no)
 		(fields_autoplaced yes)
-		(property "Reference" "R400"
+		(property "Reference" "R?"
 			(at 66.04 43.18 90)
 			(effects
@@
 				(path "/7e321a74-9d7c-485f-8c03-6a7893ec6c14/7e15107b-ac9e-4ac1-975d-b2dcf8c4df08"
 					(reference "R4")
+					(unit 1)
+				)
+				(path "/7e321a74-9d7c-485f-8c03-6a7893ec6c14/a8302038-da8a-47d3-9e0b-3649230cd28e"
+					(reference "R?")
 					(unit 1)
 				)
@@
 		(dnp no)
 		(fields_autoplaced yes)
-		(property "Reference" "#PWR04"
+		(property "Reference" "#PWR?"
 			(at 39.37 86.36 0)
 			(effects
@@
 				(path "/7e321a74-9d7c-485f-8c03-6a7893ec6c14/7e15107b-ac9e-4ac1-975d-b2dcf8c4df08"
 					(reference "#PWR0102")
+					(unit 1)
+				)
+				(path "/7e321a74-9d7c-485f-8c03-6a7893ec6c14/a8302038-da8a-47d3-9e0b-3649230cd28e"
+					(reference "#PWR?")
 					(unit 1)
 				)
@@
 		(on_board yes)
 		(dnp no)
-		(property "Reference" "#PWR09"
+		(property "Reference" "#PWR?"
 			(at 59.69 36.83 0)
 			(effects
@@
 				(path "/7e321a74-9d7c-485f-8c03-6a7893ec6c14/7e15107b-ac9e-4ac1-975d-b2dcf8c4df08"
 					(reference "#PWR0103")
+					(unit 1)
+				)
+				(path "/7e321a74-9d7c-485f-8c03-6a7893ec6c14/a8302038-da8a-47d3-9e0b-3649230cd28e"
+					(reference "#PWR?")
 					(unit 1)
 				)
@@
 		(dnp no)
 		(fields_autoplaced yes)
-		(property "Reference" "J2"
+		(property "Reference" "J?"
 			(at 39.37 30.48 0)
 			(effects
@@
 				(path "/7e321a74-9d7c-485f-8c03-6a7893ec6c14/7e15107b-ac9e-4ac1-975d-b2dcf8c4df08"
 					(reference "J3")
+					(unit 1)
+				)
+				(path "/7e321a74-9d7c-485f-8c03-6a7893ec6c14/a8302038-da8a-47d3-9e0b-3649230cd28e"
+					(reference "J?")
 					(unit 1)
 				)
@@
 		(dnp no)
 		(fields_autoplaced yes)
-		(property "Reference" "R300"
+		(property "Reference" "R?"
 			(at 66.04 35.56 90)
 			(effects
@@
 					(unit 1)
 				)
+				(path "/7e321a74-9d7c-485f-8c03-6a7893ec6c14/a8302038-da8a-47d3-9e0b-3649230cd28e"
+					(reference "R?")
+					(unit 1)
+				)
